File: Oath-66-Duo.kicad_sch (KiCad schematic)
At the start: 0 parts

Commit message: Schematic Updated
Parts:
- added D1, D10, D11, D12, D13, D14, D15, D16, D17, D18, D19, D2, D20, D21, D22, D23, D24, D25, D26, D27, D28, D29, D3, D30, D31, D32, D33, D4, D5, D6, D7, D8, D9: Diode, ScottoKeebs_Hotswap:Hotswap_MX_1.00u, symbol ScottoKeebs:Placeholder_Diode
- added S1, S10, S11, S12, S13, S14, S15, S16, S17, S18, S19, S2, S20, S22, S23, S24, S25, S26, S27, S28, S29, S3, S30, S31, S33, S4, S5, S6, S7, S8, S9: Keyswitch, ScottoKeebs_Hotswap:Hotswap_MX_1.00u, symbol ScottoKeebs:Placeholder_Keyswitch
- added S21: Keyswitch, ScottoKeebs_Hotswap:Hotswap_MX_2.00u_90deg, symbol ScottoKeebs:Placeholder_Keyswitch
- added S32: Keyswitch, ScottoKeebs_Hotswap:Hotswap_MX_2.00u, symbol ScottoKeebs:Placeholder_Keyswitch
- added U1: Arduino_Pro_Micro, ScottoKeebs_MCU:Arduino_Pro_Micro, symbol ScottoKeebs:MCU_Arduino_Pro_Micro
Connections:
- new net: D1.2 (A), S1.2
- new net: D11.2 (A), S11.2
- new net: D17.2 (A), S17.2
- new net: D3.2 (A), S3.2
- new net: D22.2 (A), S22.2
- new net: D32.2 (A), S32.2
- new net: D29.2 (A), S29.2
- new net: D10.2 (A), S10.2
- new net: D16.2 (A), S16.2
- new net: D19.2 (A), S19.2
- new net: D5.2 (A), S5.2
- new net: D20.2 (A), S20.2
- new net: D7.2 (A), S7.2
- new net: D12.2 (A), S12.2
- new net: D24.2 (A), S24.2
- new net: D9.2 (A), S9.2
- new net: D26.2 (A), S26.2
- new net: D2.2 (A), S2.2
- new net: D27.2 (A), S27.2
- new net: D33.2 (A), S33.2
- new net: D21.2 (A), S21.2
- new net: D28.2 (A), S28.2
- new net: D30.2 (A), S30.2
- new net: D18.2 (A), S18.2
- new net: D8.2 (A), S8.2
- new net: D15.2 (A), S15.2
- new net: D14.2 (A), S14.2
- new net: D13.2 (A), S13.2
- new net: D25.2 (A), S25.2
- new net: D23.2 (A), S23.2
- new net: D4.2 (A), S4.2
- new net: D31.2 (A), S31.2
- new net: D6.2 (A), S6.2
- new net Col 0: S1.1, S15.1, S22.1, S28.1, S8.1, U1.5 (2/PD1)
- new net Col 1: S16.1, S2.1, S23.1, S29.1, S9.1, U1.6 (3/PD0)
- new net Col 2: S10.1, S17.1, S24.1, S3.1, S30.1, U1.7 (4/PD4)
- new net Col 3: S11.1, S18.1, S25.1, S31.1, S4.1, U1.8 (5/PC6)
- new net Col 4: S12.1, S19.1, S26.1, S32.1, S5.1, U1.9 (6/PD7)
- new net Col 5: S13.1, S20.1, S27.1, S33.1, S6.1, U1.10 (7/PE6)
- new net Col 6: S14.1, S21.1, S7.1, U1.11 (8/PB4)
- new net Row 0: D1.1 (K), D2.1 (K), D3.1 (K), D4.1 (K), D5.1 (K), D6.1 (K), D7.1 (K), U1.12 (9/PB5)
- new net Row 1: D10.1 (K), D11.1 (K), D12.1 (K), D13.1 (K), D14.1 (K), D8.1 (K), D9.1 (K), U1.13 (10/PB6)
- new net Row 2: D15.1 (K), D16.1 (K), D17.1 (K), D18.1 (K), D19.1 (K), D20.1 (K), D21.1 (K), U1.14 (16/PB2)
- new net Row 3: D22.1 (K), D23.1 (K), D24.1 (K), D25.1 (K), D26.1 (K), D27.1 (K), U1.15 (14/PB3)
- new net Row 4: D28.1 (K), D29.1 (K), D30.1 (K), D31.1 (K), D32.1 (K), D33.1 (K), U1.16 (15/PB1)

Commit message: PCB Updated
Parts:
- D1, D10, D11, D12, D13, D14, D15, D16, D17, D18, D19, D2, D20, D21, D22, D23, D24, D25, D26, D27, D28, D29, D3, D30, D31, D32, D33, D4, D5, D6, D7, D8, D9: footprint ScottoKeebs_Hotswap:Hotswap_MX_1.00u -> ScottoKeebs_Components:Diode_SOD-123
Changed lines of the file:
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@@
 			)
 		)
-		(property "Footprint" "ScottoKeebs_Hotswap:Hotswap_MX_1.00u"
+		(property "Footprint" "ScottoKeebs_Components:Diode_SOD-123"
 			(at 34.29 50.8 0)
 			(effects
@@
 			)
 		)
-		(property "Footprint" "ScottoKeebs_Hotswap:Hotswap_MX_1.00u"
+		(property "Footprint" "ScottoKeebs_Components:Diode_SOD-123"
 			(at 68.58 71.12 0)
 			(effects
@@
 			)
 		)
-		(property "Footprint" "ScottoKeebs_Hotswap:Hotswap_MX_1.00u"
+		(property "Footprint" "ScottoKeebs_Components:Diode_SOD-123"
 			(at 57.15 50.8 0)
 			(effects
@@
 			)
 		)
-		(property "Footprint" "ScottoKeebs_Hotswap:Hotswap_MX_1.00u"
+		(property "Footprint" "ScottoKeebs_Components:Diode_SOD-123"
 			(at 57.15 71.12 0)
 			(effects
@@
 			)
 		)
-		(property "Footprint" "ScottoKeebs_Hotswap:Hotswap_MX_1.00u"
+		(property "Footprint" "ScottoKeebs_Components:Diode_SOD-123"
 			(at 91.44 91.44 0)
 			(effects
@@
 			)
 		)
-		(property "Footprint" "ScottoKeebs_Hotswap:Hotswap_MX_1.00u"
+		(property "Footprint" "ScottoKeebs_Components:Diode_SOD-123"
 			(at 80.01 132.08 0)
 			(effects
@@
 			)
 		)
-		(property "Footprint" "ScottoKeebs_Hotswap:Hotswap_MX_1.00u"
+		(property "Footprint" "ScottoKeebs_Components:Diode_SOD-123"
 			(at 102.87 50.8 0)
 			(effects
@@
 			)
 		)
-		(property "Footprint" "ScottoKeebs_Hotswap:Hotswap_MX_1.00u"
+		(property "Footprint" "ScottoKeebs_Components:Diode_SOD-123"
 			(at 80.01 71.12 0)
 			(effects
@@
 			)
 		)
-		(property "Footprint" "ScottoKeebs_Hotswap:Hotswap_MX_1.00u"
+		(property "Footprint" "ScottoKeebs_Components:Diode_SOD-123"
 			(at 57.15 111.76 0)
 			(effects
@@
 			)
 		)
-		(property "Footprint" "ScottoKeebs_Hotswap:Hotswap_MX_1.00u"
+		(property "Footprint" "ScottoKeebs_Components:Diode_SOD-123"
 			(at 80.01 50.8 0)
 			(effects
@@
 			)
 		)
-		(property "Footprint" "ScottoKeebs_Hotswap:Hotswap_MX_1.00u"
+		(property "Footprint" "ScottoKeebs_Components:Diode_SOD-123"
 			(at 57.15 91.44 0)
 			(effects
@@
 			)
 		)
-		(property "Footprint" "ScottoKeebs_Hotswap:Hotswap_MX_1.00u"
+		(property "Footprint" "ScottoKeebs_Components:Diode_SOD-123"
 			(at 80.01 111.76 0)
 			(effects
@@
 			)
 		)
-		(property "Footprint" "ScottoKeebs_Hotswap:Hotswap_MX_1.00u"
+		(property "Footprint" "ScottoKeebs_Components:Diode_SOD-123"
 			(at 102.87 91.44 0)
 			(effects
@@
 			)
 		)
-		(property "Footprint" "ScottoKeebs_Hotswap:Hotswap_MX_1.00u"
+		(property "Footprint" "ScottoKeebs_Components:Diode_SOD-123"
 			(at 34.29 132.08 0)
 			(effects
@@
 			)
 		)
-		(property "Footprint" "ScottoKeebs_Hotswap:Hotswap_MX_1.00u"
+		(property "Footprint" "ScottoKeebs_Components:Diode_SOD-123"
 			(at 57.15 132.08 0)
 			(effects
@@
 			)
 		)
-		(property "Footprint" "ScottoKeebs_Hotswap:Hotswap_MX_1.00u"
+		(property "Footprint" "ScottoKeebs_Components:Diode_SOD-123"
 			(at 68.58 91.44 0)
 			(effects
@@
 			)
 		)
-		(property "Footprint" "ScottoKeebs_Hotswap:Hotswap_MX_1.00u"
+		(property "Footprint" "ScottoKeebs_Components:Diode_SOD-123"
 			(at 34.29 71.12 0)
 			(effects
@@
 			)
 		)
-		(property "Footprint" "ScottoKeebs_Hotswap:Hotswap_MX_1.00u"
+		(property "Footprint" "ScottoKeebs_Components:Diode_SOD-123"
 			(at 34.29 91.44 0)
 			(effects
@@
 			)
 		)
-		(property "Footprint" "ScottoKeebs_Hotswap:Hotswap_MX_1.00u"
+		(property "Footprint" "ScottoKeebs_Components:Diode_SOD-123"
 			(at 45.72 91.44 0)
 			(effects
@@
 			)
 		)
-		(property "Footprint" "ScottoKeebs_Hotswap:Hotswap_MX_1.00u"
+		(property "Footprint" "ScottoKeebs_Components:Diode_SOD-123"
 			(at 45.72 132.08 0)
 			(effects
@@
 			)
 		)
-		(property "Footprint" "ScottoKeebs_Hotswap:Hotswap_MX_1.00u"
+		(property "Footprint" "ScottoKeebs_Components:Diode_SOD-123"
 			(at 45.72 71.12 0)
 			(effects
@@
 			)
 		)
-		(property "Footprint" "ScottoKeebs_Hotswap:Hotswap_MX_1.00u"
+		(property "Footprint" "ScottoKeebs_Components:Diode_SOD-123"
 			(at 102.87 71.12 0)
 			(effects
@@
 			)
 		)
-		(property "Footprint" "ScottoKeebs_Hotswap:Hotswap_MX_1.00u"
+		(property "Footprint" "ScottoKeebs_Components:Diode_SOD-123"
 			(at 91.44 71.12 0)
 			(effects
@@
 			)
 		)
-		(property "Footprint" "ScottoKeebs_Hotswap:Hotswap_MX_1.00u"
+		(property "Footprint" "ScottoKeebs_Components:Diode_SOD-123"
 			(at 68.58 111.76 0)
 			(effects
@@
 			)
 		)
-		(property "Footprint" "ScottoKeebs_Hotswap:Hotswap_MX_1.00u"
+		(property "Footprint" "ScottoKeebs_Components:Diode_SOD-123"
 			(at 80.01 91.44 0)
 			(effects
@@
 			)
 		)
-		(property "Footprint" "ScottoKeebs_Hotswap:Hotswap_MX_1.00u"
+		(property "Footprint" "ScottoKeebs_Components:Diode_SOD-123"
 			(at 91.44 111.76 0)
 			(effects
@@
 			)
 		)
-		(property "Footprint" "ScottoKeebs_Hotswap:Hotswap_MX_1.00u"
+		(property "Footprint" "ScottoKeebs_Components:Diode_SOD-123"
 			(at 34.29 111.76 0)
 			(effects
@@
 			)
 		)
-		(property "Footprint" "ScottoKeebs_Hotswap:Hotswap_MX_1.00u"
+		(property "Footprint" "ScottoKeebs_Components:Diode_SOD-123"
 			(at 68.58 50.8 0)
 			(effects
@@
 			)
 		)
-		(property "Footprint" "ScottoKeebs_Hotswap:Hotswap_MX_1.00u"
+		(property "Footprint" "ScottoKeebs_Components:Diode_SOD-123"
 			(at 91.44 50.8 0)
 			(effects
@@
 			)
 		)
-		(property "Footprint" "ScottoKeebs_Hotswap:Hotswap_MX_1.00u"
+		(property "Footprint" "ScottoKeebs_Components:Diode_SOD-123"
 			(at 91.44 132.08 0)
 			(effects
@@
 			)
 		)
-		(property "Footprint" "ScottoKeebs_Hotswap:Hotswap_MX_1.00u"
+		(property "Footprint" "ScottoKeebs_Components:Diode_SOD-123"
 			(at 45.72 111.76 0)
 			(effects
@@
 			)
 		)
-		(property "Footprint" "ScottoKeebs_Hotswap:Hotswap_MX_1.00u"
+		(property "Footprint" "ScottoKeebs_Components:Diode_SOD-123"
 			(at 68.58 132.08 0)
 			(effects
@@
 			)
 		)
-		(property "Footprint" "ScottoKeebs_Hotswap:Hotswap_MX_1.00u"
+		(property "Footprint" "ScottoKeebs_Components:Diode_SOD-123"
 			(at 45.72 50.8 0)
 			(effects

Commit message: Schematic and PVB updated
Parts:
- renumbered D22 to D21, D23 to D22, D24 to D23, D25 to D24, D26 to D25, D27 to D26, D21 to D27, S22 to S21, S23 to S22, S24 to S23, S25 to S24, S26 to S25, S27 to S26, S21 to S27
Connections:
- net Col 0: now also U1.8 (5/PC6); no longer U1.5 (2/PD1)
- net Col 1: now also U1.10 (7/PE6); no longer U1.6 (3/PD0)
- net Col 2: now also U1.11 (8/PB4); no longer U1.7 (4/PD4)
- net Col 3: now also U1.15 (14/PB3); no longer U1.8 (5/PC6)
- net Col 4: now also U1.13 (10/PB6); no longer U1.9 (6/PD7)
- net Col 5: now also U1.5 (2/PD1); no longer S33.1, U1.10 (7/PE6)
- net Col 6: now also S33.1, U1.6 (3/PD0); no longer U1.11 (8/PB4)
- net Row 0: now also U1.7 (4/PD4); no longer U1.12 (9/PB5)
- net Row 1: now also U1.9 (6/PD7); no longer U1.13 (10/PB6)
- net Row 2: now also U1.12 (9/PB5); no longer D27.1 (K), U1.14 (16/PB2)
- net Row 3: now also D27.1 (K), U1.16 (15/PB1); no longer U1.15 (14/PB3)
- net Row 4: now also U1.14 (16/PB2); no longer U1.16 (15/PB1)
Other:
- moved on the sheet: D27, D33, S27, S33

Commit message: Sub-Schematic Updated
Parts:
- removed D1, D10, D11, D12, D13, D14, D15, D16, D17, D18, D19, D2, D20, D21, D22, D23, D24, D25, D26, D27, D28, D29, D3, D30, D31, D32, D33, D4, D5, D6, D7, D8, D9: Diode, ScottoKeebs_Components:Diode_SOD-123, symbol ScottoKeebs:Placeholder_Diode
- removed S1, S10, S11, S12, S13, S14, S15, S16, S17, S18, S19, S2, S20, S21, S22, S23, S24, S25, S26, S28, S29, S3, S30, S31, S33, S4, S5, S6, S7, S8, S9: Keyswitch, ScottoKeebs_Hotswap:Hotswap_MX_1.00u, symbol ScottoKeebs:Placeholder_Keyswitch
- removed S27: Keyswitch, ScottoKeebs_Hotswap:Hotswap_MX_2.00u_90deg, symbol ScottoKeebs:Placeholder_Keyswitch
- removed S32: Keyswitch, ScottoKeebs_Hotswap:Hotswap_MX_2.00u, symbol ScottoKeebs:Placeholder_Keyswitch
- removed U1: Arduino_Pro_Micro, ScottoKeebs_MCU:Arduino_Pro_Micro, symbol ScottoKeebs:MCU_Arduino_Pro_Micro
Other:
- added sheet Oath-66-Duo-Dongle (Oath-66-Duo-Dongle.kicad_sch)
- added sheet Oath-66-Duo-Left (Oath-66-Duo-Left.kicad_sch)
- added sheet Oath-66-Duo-Right (Oath-66-Duo-Right.kicad_sch)
