File: Oath-66-Duo-Left.kicad_sch (KiCad schematic)
At the start: 67 parts, among them U1 Arduino_Pro_Micro

Commit message: PCB Updated
Parts:
- S15, S21, S8: footprint ScottoKeebs_Hotswap:Hotswap_MX_1.00u -> ScottoKeebs_Hotswap:Hotswap_MX_1.50u
Changed lines of the file:
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@@
 			)
 		)
-		(property "Footprint" "ScottoKeebs_Hotswap:Hotswap_MX_1.00u"
+		(property "Footprint" "ScottoKeebs_Hotswap:Hotswap_MX_1.50u"
 			(at 191.77 111.76 0)
 			(effects
@@
 			)
 		)
-		(property "Footprint" "ScottoKeebs_Hotswap:Hotswap_MX_1.00u"
+		(property "Footprint" "ScottoKeebs_Hotswap:Hotswap_MX_1.50u"
 			(at 191.77 91.44 0)
 			(effects
@@
 			)
 		)
-		(property "Footprint" "ScottoKeebs_Hotswap:Hotswap_MX_1.00u"
+		(property "Footprint" "ScottoKeebs_Hotswap:Hotswap_MX_1.50u"
 			(at 191.77 71.12 0)
 			(effects
