File: Oath-66-Duo-Right.kicad_sch (KiCad schematic)
At the start: 67 parts, among them U2 Arduino_Pro_Micro

Commit message: PCB Updated
Parts:
- renumbered D49 to D48, D50 to D49, D51 to D50, D52 to D51, D53 to D52, D48 to D53, S49 to S48, S50 to S49, S51 to S50, S52 to S51, S53 to S52, S48 to S53
Connections:
- net Row 2 is gone; now on net Col 0: D48.1 (K), D49.1 (K), D50.1 (K), D51.1 (K), D52.1 (K), D53.1 (K), U2.12 (9/PB5)
- net Col 0: no longer S53.1
- net Col 1: no longer S62.1
- net Col 2: now also S62.1; no longer S63.1
- net Col 3: now also S63.1; no longer S64.1
- net Col 4: now also S64.1; no longer S65.1
- net Col 5: now also S65.1
- net Col 6: now also S53.1
Other:
- moved on the sheet: D53, D62, D63, D64, D65, S53, S62, S63, S64, S65

Commit message: PCB Updated
Parts:
- S47, S52: footprint ScottoKeebs_Hotswap:Hotswap_MX_1.00u -> ScottoKeebs_Hotswap:Hotswap_MX_1.50u
- S54: footprint ScottoKeebs_Hotswap:Hotswap_MX_1.00u -> ScottoKeebs_Hotswap:Hotswap_MX_2.00u_90deg
- S60: footprint ScottoKeebs_Hotswap:Hotswap_MX_2.00u_90deg -> ScottoKeebs_Hotswap:Hotswap_MX_1.50u
- S62: footprint ScottoKeebs_Hotswap:Hotswap_MX_1.00u -> ScottoKeebs_Hotswap:Hotswap_MX_2.00u
- S65: footprint ScottoKeebs_Hotswap:Hotswap_MX_2.00u -> ScottoKeebs_Hotswap:Hotswap_MX_1.00u
Changed lines of the file:
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@@
 			)
 		)
-		(property "Footprint" "ScottoKeebs_Hotswap:Hotswap_MX_1.00u"
+		(property "Footprint" "ScottoKeebs_Hotswap:Hotswap_MX_2.00u_90deg"
 			(at 191.77 111.76 0)
 			(effects
@@
 			)
 		)
-		(property "Footprint" "ScottoKeebs_Hotswap:Hotswap_MX_2.00u_90deg"
+		(property "Footprint" "ScottoKeebs_Hotswap:Hotswap_MX_1.50u"
 			(at 260.35 111.76 0)
 			(effects
@@
 			)
 		)
-		(property "Footprint" "ScottoKeebs_Hotswap:Hotswap_MX_1.00u"
+		(property "Footprint" "ScottoKeebs_Hotswap:Hotswap_MX_2.00u"
 			(at 214.63 132.08 0)
 			(effects
@@
 			)
 		)
-		(property "Footprint" "ScottoKeebs_Hotswap:Hotswap_MX_1.00u"
+		(property "Footprint" "ScottoKeebs_Hotswap:Hotswap_MX_1.50u"
 			(at 260.35 71.12 0)
 			(effects
@@
 			)
 		)
-		(property "Footprint" "ScottoKeebs_Hotswap:Hotswap_MX_1.00u"
+		(property "Footprint" "ScottoKeebs_Hotswap:Hotswap_MX_1.50u"
 			(at 248.92 91.44 0)
 			(effects
@@
 			)
 		)
-		(property "Footprint" "ScottoKeebs_Hotswap:Hotswap_MX_2.00u"
+		(property "Footprint" "ScottoKeebs_Hotswap:Hotswap_MX_1.00u"
 			(at 248.92 132.08 0)
 			(effects
