File: Oath-66-Duo.kicad_pcb (KiCad board)
At the start: 2 copper layers, 67 parts, among them U1 Arduino_Pro_Micro

Commit message: Schematic and PVB updated
Parts:
- added REF**: MountingHole_2.5mm, MountingHole:MountingHole_2.5mm, F.Cu at (26.0, 27.0)
- added REF**: MountingHole_2.5mm, MountingHole:MountingHole_2.5mm, F.Cu at (26.0, 125.5)
- added REF**: MountingHole_2.5mm, MountingHole:MountingHole_2.5mm, F.Cu at (188.5, 27.0)
- added REF**: MountingHole_2.5mm, MountingHole:MountingHole_2.5mm, F.Cu at (188.5, 125.5)
- moved U1 5.32 mm to (176.2, 42.9)
- renumbered D22 to D21, D23 to D22, D24 to D23, D25 to D24, D26 to D25, D27 to D26, D21 to D27, S22 to S21, S23 to S22, S24 to S23, S25 to S24, S26 to S25, S27 to S26, S21 to S27
Connections:
- D27 pad 1: Row 2 -> Row 3
- S33 pad 1: Col 5 -> Col 6
- U1 pad 10: Col 5 -> Col 1
- U1 pad 11: Col 6 -> Col 2
- U1 pad 12: Row 0 -> Row 2
- U1 pad 13: Row 1 -> Col 4
- U1 pad 14: Row 2 -> Row 4
- U1 pad 15: Row 3 -> Col 3
- U1 pad 16: Row 4 -> Row 3
- U1 pad 5: Col 0 -> Col 5
- U1 pad 6: Col 1 -> Col 6
- U1 pad 7: Col 2 -> Row 0
- U1 pad 8: Col 3 -> Col 0
- U1 pad 9: Col 4 -> Row 1
Routing:
- net Col 4: track 0.00 -> 240.5 mm, vias 0 -> 2
- net Col 3: track 0.00 -> 221.8 mm, vias 0 -> 2
- net Row 4: track 0.00 -> 219.0 mm, vias 0 -> 7
- net Col 2: track 0.00 -> 216.5 mm, vias 0 -> 2
- net Col 0: track 0.00 -> 214.3 mm, vias 0 -> 1
- net Row 3: track 0.00 -> 207.9 mm, vias 0 -> 8
- net Col 1: track 0.00 -> 205.7 mm, vias 0 -> 1
- net Row 2: track 0.00 -> 159.9 mm, vias 0 -> 6
- net Row 1: track 0.00 -> 153.9 mm, vias 0 -> 7
- net Row 0: track 0.00 -> 143.2 mm, vias 0 -> 7
- net Col 5: track 0.00 -> 111.7 mm
- net Col 6: track 0.00 -> 109.5 mm
- net Net-(D27-A): track 0.00 -> 16.9 mm
- net Net-(D32-A): track 0.00 -> 15.6 mm
- net Net-(D14-A): track 0.00 -> 7.34 mm
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- added copper zone on B.Cu, net (none)
- added copper zone on F.Cu, net (none)
Other:
- board outline added: 168.5 x 104.5 mm

Commit message: Sub-Schematic Updated
Parts:
- removed REF** (x4): MountingHole_2.5mm, MountingHole:MountingHole_2.5mm
- added D34: Diode, ScottoKeebs_Components:Diode_SOD-123, F.Cu at (374.9, 62.4)
- added D35: Diode, ScottoKeebs_Components:Diode_SOD-123, F.Cu at (374.9, 65.8)
- added D36: Diode, ScottoKeebs_Components:Diode_SOD-123, F.Cu at (374.9, 69.1)
- added D37: Diode, ScottoKeebs_Components:Diode_SOD-123, F.Cu at (374.9, 72.5)
- added D38: Diode, ScottoKeebs_Components:Diode_SOD-123, F.Cu at (374.9, 75.8)
- added D39: Diode, ScottoKeebs_Components:Diode_SOD-123, F.Cu at (374.9, 79.2)
- added D40: Diode, ScottoKeebs_Components:Diode_SOD-123, F.Cu at (374.9, 82.5)
- added D41: Diode, ScottoKeebs_Components:Diode_SOD-123, F.Cu at (374.9, 85.9)
- added D42: Diode, ScottoKeebs_Components:Diode_SOD-123, F.Cu at (374.9, 89.2)
- added D43: Diode, ScottoKeebs_Components:Diode_SOD-123, F.Cu at (380.7, 62.4)
- added D44: Diode, ScottoKeebs_Components:Diode_SOD-123, F.Cu at (380.7, 65.8)
- added D45: Diode, ScottoKeebs_Components:Diode_SOD-123, F.Cu at (380.7, 69.1)
- added D46: Diode, ScottoKeebs_Components:Diode_SOD-123, F.Cu at (380.7, 72.5)
- added D47: Diode, ScottoKeebs_Components:Diode_SOD-123, F.Cu at (380.7, 75.8)
- added D48: Diode, ScottoKeebs_Components:Diode_SOD-123, F.Cu at (380.7, 79.2)
- added D49: Diode, ScottoKeebs_Components:Diode_SOD-123, F.Cu at (380.7, 82.5)
- added D50: Diode, ScottoKeebs_Components:Diode_SOD-123, F.Cu at (380.7, 85.9)
- added D51: Diode, ScottoKeebs_Components:Diode_SOD-123, F.Cu at (380.7, 89.2)
- added D52: Diode, ScottoKeebs_Components:Diode_SOD-123, F.Cu at (386.4, 62.4)
- added D53: Diode, ScottoKeebs_Components:Diode_SOD-123, F.Cu at (386.4, 65.8)
- added D54: Diode, ScottoKeebs_Components:Diode_SOD-123, F.Cu at (386.4, 69.1)
- added D55: Diode, ScottoKeebs_Components:Diode_SOD-123, F.Cu at (386.4, 72.5)
- added D56: Diode, ScottoKeebs_Components:Diode_SOD-123, F.Cu at (386.4, 75.8)
- added D57: Diode, ScottoKeebs_Components:Diode_SOD-123, F.Cu at (386.4, 79.2)
- added D58: Diode, ScottoKeebs_Components:Diode_SOD-123, F.Cu at (386.4, 82.5)
- added D59: Diode, ScottoKeebs_Components:Diode_SOD-123, F.Cu at (386.4, 85.9)
- added D60: Diode, ScottoKeebs_Components:Diode_SOD-123, F.Cu at (386.4, 89.2)
- added D61: Diode, ScottoKeebs_Components:Diode_SOD-123, F.Cu at (392.2, 62.4)
- added D62: Diode, ScottoKeebs_Components:Diode_SOD-123, F.Cu at (392.2, 65.8)
- added D63: Diode, ScottoKeebs_Components:Diode_SOD-123, F.Cu at (392.2, 69.1)
- added D64: Diode, ScottoKeebs_Components:Diode_SOD-123, F.Cu at (392.2, 72.5)
- added D65: Diode, ScottoKeebs_Components:Diode_SOD-123, F.Cu at (392.2, 75.8)
- added D66: Diode, ScottoKeebs_Components:Diode_SOD-123, F.Cu at (392.2, 79.2)
- added S34: Keyswitch, ScottoKeebs_Hotswap:Hotswap_MX_1.00u, F.Cu at (297.8, 34.3)
- added S35: Keyswitch, ScottoKeebs_Hotswap:Hotswap_MX_1.00u, F.Cu at (297.8, 49.9)
- added S36: Keyswitch, ScottoKeebs_Hotswap:Hotswap_MX_1.00u, F.Cu at (297.8, 65.4)
- added S37: Keyswitch, ScottoKeebs_Hotswap:Hotswap_MX_1.00u, F.Cu at (297.8, 81.0)
- added S38: Keyswitch, ScottoKeebs_Hotswap:Hotswap_MX_1.00u, F.Cu at (297.8, 96.5)
- added S39: Keyswitch, ScottoKeebs_Hotswap:Hotswap_MX_1.00u, F.Cu at (297.8, 112.1)
- added S40: Keyswitch, ScottoKeebs_Hotswap:Hotswap_MX_1.00u, F.Cu at (297.8, 127.6)
- added S41: Keyswitch, ScottoKeebs_Hotswap:Hotswap_MX_1.00u, F.Cu at (314.4, 34.3)
- added S42: Keyswitch, ScottoKeebs_Hotswap:Hotswap_MX_1.00u, F.Cu at (314.4, 49.9)
- added S43: Keyswitch, ScottoKeebs_Hotswap:Hotswap_MX_1.00u, F.Cu at (314.4, 65.4)
- added S44: Keyswitch, ScottoKeebs_Hotswap:Hotswap_MX_1.00u, F.Cu at (314.4, 81.0)
- added S45: Keyswitch, ScottoKeebs_Hotswap:Hotswap_MX_1.00u, F.Cu at (314.4, 96.5)
- added S46: Keyswitch, ScottoKeebs_Hotswap:Hotswap_MX_1.00u, F.Cu at (314.4, 112.1)
- added S47: Keyswitch, ScottoKeebs_Hotswap:Hotswap_MX_1.00u, F.Cu at (314.4, 127.6)
- added S48: Keyswitch, ScottoKeebs_Hotswap:Hotswap_MX_1.00u, F.Cu at (331.0, 34.3)
- added S49: Keyswitch, ScottoKeebs_Hotswap:Hotswap_MX_1.00u, F.Cu at (331.0, 49.9)
- added S50: Keyswitch, ScottoKeebs_Hotswap:Hotswap_MX_1.00u, F.Cu at (331.0, 65.4)
- added S51: Keyswitch, ScottoKeebs_Hotswap:Hotswap_MX_1.00u, F.Cu at (331.0, 81.0)
- added S52: Keyswitch, ScottoKeebs_Hotswap:Hotswap_MX_1.00u, F.Cu at (331.0, 96.5)
- added S53: Keyswitch, ScottoKeebs_Hotswap:Hotswap_MX_1.00u, F.Cu at (331.0, 112.1)
- added S54: Keyswitch, ScottoKeebs_Hotswap:Hotswap_MX_1.00u, F.Cu at (331.0, 127.6)
- added S55: Keyswitch, ScottoKeebs_Hotswap:Hotswap_MX_1.00u, F.Cu at (347.7, 34.3)
- added S56: Keyswitch, ScottoKeebs_Hotswap:Hotswap_MX_1.00u, F.Cu at (347.7, 49.9)
- added S57: Keyswitch, ScottoKeebs_Hotswap:Hotswap_MX_1.00u, F.Cu at (347.7, 65.4)
- added S58: Keyswitch, ScottoKeebs_Hotswap:Hotswap_MX_1.00u, F.Cu at (347.7, 81.0)
- added S59: Keyswitch, ScottoKeebs_Hotswap:Hotswap_MX_1.00u, F.Cu at (347.7, 96.5)
- added S60: Keyswitch, ScottoKeebs_Hotswap:Hotswap_MX_2.00u_90deg, F.Cu at (347.7, 112.1)
- added S61: Keyswitch, ScottoKeebs_Hotswap:Hotswap_MX_1.00u, F.Cu at (347.7, 127.6)
- added S62: Keyswitch, ScottoKeebs_Hotswap:Hotswap_MX_1.00u, F.Cu at (364.3, 34.3)
- added S63: Keyswitch, ScottoKeebs_Hotswap:Hotswap_MX_1.00u, F.Cu at (364.3, 49.9)
- added S64: Keyswitch, ScottoKeebs_Hotswap:Hotswap_MX_1.00u, F.Cu at (364.3, 65.4)
- added S65: Keyswitch, ScottoKeebs_Hotswap:Hotswap_MX_2.00u, F.Cu at (364.3, 81.0)
- added S66: Keyswitch, ScottoKeebs_Hotswap:Hotswap_MX_1.00u, F.Cu at (364.3, 96.5)
- added U2: Arduino_Pro_Micro, ScottoKeebs_MCU:Arduino_Pro_Micro, F.Cu at (381.6, 44.9)
- D1, D10, D11, D12, D13, D14, D15, D16, D17, D18, D19, D2, D20, D21, D22, D23, D24, D25, D26, D27, D28, D29, D3, D30, D31, D32, D33, D4, D5, D6, D7, D8, D9: moved to F.Cu
- moved S7 143.3 mm to (46.8, 134.9)
- moved S6 118.7 mm to (46.8, 119.4)
- moved S14 118.2 mm to (63.4, 134.9)
- moved D28 104.7 mm to (141.2, 69.7), turned to 0 degrees
- moved S5 94.2 mm to (46.8, 103.8)
- moved S13 93.6 mm to (63.4, 119.4)
- moved S29 91.9 mm to (113.3, 41.6)
- moved D21 90.4 mm to (135.5, 76.4), turned to 0 degrees
- moved D29 86.3 mm to (141.2, 73.1), turned to 0 degrees
- moved D8 83.4 mm to (124.0, 93.2), turned to 0 degrees
- moved D15 82.5 mm to (129.7, 86.5), turned to 0 degrees
- moved D1 81.7 mm to (124.0, 69.7), turned to 0 degrees
- moved D22 71.1 mm to (135.5, 79.8), turned to 0 degrees
- moved S4 69.8 mm to (46.8, 88.3)
- moved S12 69.0 mm to (63.4, 103.8)
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Connections:
- net Col 0 renamed /Oath-66-Duo-Left/Col 0
- net Col 1 renamed /Oath-66-Duo-Left/Col 1
- net Col 2 renamed /Oath-66-Duo-Left/Col 2
- net Col 3 renamed /Oath-66-Duo-Left/Col 3
- net Col 4 renamed /Oath-66-Duo-Left/Col 4
- net Col 5 renamed /Oath-66-Duo-Left/Col 5
- net Col 6 renamed /Oath-66-Duo-Left/Col 6
- net Row 0 renamed /Oath-66-Duo-Left/Row 0
- net Row 1 renamed /Oath-66-Duo-Left/Row 1
- net Row 2 renamed /Oath-66-Duo-Left/Row 2
- net Row 3 renamed /Oath-66-Duo-Left/Row 3
- net Row 4 renamed /Oath-66-Duo-Left/Row 4
Routing:
- net /Oath-66-Duo-Left/Col 4: track 240.5 -> 0.00 mm, vias 2 -> 0
- net /Oath-66-Duo-Left/Col 3: track 221.8 -> 0.00 mm, vias 2 -> 0
- net /Oath-66-Duo-Left/Row 4: track 219.0 -> 0.00 mm, vias 7 -> 0
- net /Oath-66-Duo-Left/Col 2: track 216.5 -> 0.00 mm, vias 2 -> 0
- net /Oath-66-Duo-Left/Col 0: track 214.3 -> 0.00 mm, vias 1 -> 0
- net /Oath-66-Duo-Left/Row 3: track 207.9 -> 0.00 mm, vias 8 -> 0
- net /Oath-66-Duo-Left/Col 1: track 205.7 -> 0.00 mm, vias 1 -> 0
- net /Oath-66-Duo-Left/Row 2: track 159.9 -> 0.00 mm, vias 6 -> 0
- net /Oath-66-Duo-Left/Row 1: track 153.9 -> 0.00 mm, vias 7 -> 0
- net /Oath-66-Duo-Left/Row 0: track 143.2 -> 0.00 mm, vias 7 -> 0
- net /Oath-66-Duo-Left/Col 5: track 111.7 -> 0.00 mm
- net /Oath-66-Duo-Left/Col 6: track 109.5 -> 0.00 mm
- net Net-(D27-A): track 16.9 -> 0.00 mm
- net Net-(D32-A): track 15.6 -> 0.00 mm
- net Net-(D14-A): track 7.34 -> 0.00 mm
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- removed copper zone on B.Cu, net (none)
- removed copper zone on F.Cu, net (none)
Other:
- board outline removed

Commit message: PCB Updated
Parts:
- S15, S21, S8: footprint ScottoKeebs_Hotswap:Hotswap_MX_1.00u -> ScottoKeebs_Hotswap:Hotswap_MX_1.50u
- U1: moved to B.Cu
- moved S7 158.9 mm to (172.8, 38.1)
- moved S6 134.3 mm to (153.7, 38.1)
- moved S14 134.2 mm to (172.8, 57.1)
- moved D1 115.6 mm to (238.5, 54.2)
- moved D2 115.6 mm to (238.5, 57.6)
- moved D3 115.6 mm to (238.5, 60.9)
- moved D4 115.6 mm to (238.5, 64.3)
- moved D5 115.6 mm to (238.5, 67.6)
- moved D6 115.6 mm to (238.5, 71.0)
- moved D7 115.6 mm to (238.5, 74.3)
- moved D8 115.6 mm to (238.5, 77.7)
- moved D9 115.6 mm to (238.5, 81.0)
- moved D10 115.6 mm to (244.3, 54.2)
- moved D11 115.6 mm to (244.3, 57.6)
- moved D12 115.6 mm to (244.3, 60.9)
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
Commit message: PCB Updated
Parts:
- S47: footprint ScottoKeebs_Hotswap:Hotswap_MX_1.00u -> ScottoKeebs_Hotswap:Hotswap_MX_1.50u
- S52: renamed from S53; footprint ScottoKeebs_Hotswap:Hotswap_MX_1.00u -> ScottoKeebs_Hotswap:Hotswap_MX_1.50u
- S54: footprint ScottoKeebs_Hotswap:Hotswap_MX_1.00u -> ScottoKeebs_Hotswap:Hotswap_MX_2.00u_90deg
- S60: footprint ScottoKeebs_Hotswap:Hotswap_MX_2.00u_90deg -> ScottoKeebs_Hotswap:Hotswap_MX_1.50u
- S62: footprint ScottoKeebs_Hotswap:Hotswap_MX_1.00u -> ScottoKeebs_Hotswap:Hotswap_MX_2.00u
- S65: footprint ScottoKeebs_Hotswap:Hotswap_MX_2.00u -> ScottoKeebs_Hotswap:Hotswap_MX_1.00u
- moved D1 137.0 mm to (139.4, 148.9)
- moved D10 137.0 mm to (145.2, 148.9)
- moved D11 137.0 mm to (145.2, 152.2)
- moved D12 137.0 mm to (145.2, 155.6)
- moved D13 137.0 mm to (145.2, 158.9)
- moved D14 137.0 mm to (145.2, 162.3)
- moved D15 137.0 mm to (145.2, 165.6)
- moved D16 137.0 mm to (145.2, 169.0)
- moved D17 137.0 mm to (145.2, 172.3)
- moved D18 137.0 mm to (145.2, 175.7)
- moved D19 137.0 mm to (150.9, 148.9)
- moved D2 137.0 mm to (139.4, 152.2)
- moved D20 137.0 mm to (150.9, 152.2)
- moved D21 137.0 mm to (150.9, 155.6)
- moved D22 137.0 mm to (150.9, 158.9)
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- renumbered D49 to D48, D50 to D49, D51 to D50, D52 to D51, D53 to D52, D48 to D53, S49 to S48, S50 to S49, S51 to S50, S52 to S51, S48 to S53
Connections:
- D48 pad 1: /Oath-66-Duo-Right/Row 2 -> /Oath-66-Duo-Right/Col 0
- D49 pad 1: /Oath-66-Duo-Right/Row 2 -> /Oath-66-Duo-Right/Col 0
- D50 pad 1: /Oath-66-Duo-Right/Row 2 -> /Oath-66-Duo-Right/Col 0
- D51 pad 1: /Oath-66-Duo-Right/Row 2 -> /Oath-66-Duo-Right/Col 0
- D52 pad 1: /Oath-66-Duo-Right/Row 2 -> /Oath-66-Duo-Right/Col 0
- D53 pad 1: /Oath-66-Duo-Right/Row 2 -> /Oath-66-Duo-Right/Col 0
- S53 pad 1: /Oath-66-Duo-Right/Col 0 -> /Oath-66-Duo-Right/Col 6
- S62 pad 1: /Oath-66-Duo-Right/Col 1 -> /Oath-66-Duo-Right/Col 2
- S63 pad 1: /Oath-66-Duo-Right/Col 2 -> /Oath-66-Duo-Right/Col 3
- S64 pad 1: /Oath-66-Duo-Right/Col 3 -> /Oath-66-Duo-Right/Col 4
- S65 pad 1: /Oath-66-Duo-Right/Col 4 -> /Oath-66-Duo-Right/Col 5
- U2 pad 12: /Oath-66-Duo-Right/Row 2 -> /Oath-66-Duo-Right/Col 0
