File: PCB/Oath-66-Duo.kicad_pcb (KiCad board)
At the start: 2 copper layers, 134 parts, among them U1 Arduino_Pro_Micro, U2 Arduino_Pro_Micro

Commit message: PCB Updated
Parts:
- added REF**: Stabilizer_MX_2.00u, ScottoKeebs_Stabilizer:Stabilizer_MX_2.00u, F.Cu at (181.0, 81.0)
- added REF**: Stabilizer_MX_2.00u, ScottoKeebs_Stabilizer:Stabilizer_MX_2.00u, F.Cu at (247.6, 81.0)
- added REF**: Stabilizer_MX_2.00u, ScottoKeebs_Stabilizer:Stabilizer_MX_2.00u, F.Cu at (276.2, 109.5)
- added REF**: Stabilizer_MX_2.00u, ScottoKeebs_Stabilizer:Stabilizer_MX_2.00u, F.Cu at (152.4, 109.5)
- D1, D10, D11, D12, D13, D14, D15, D16, D17, D18, D19, D2, D20, D21, D22, D23, D24, D25, D26, D27, D28, D29, D3, D30, D31, D32, D33, D34, D35, D36, D37, D38, D39, D4, D40, D41, D42, D43, D44, D45, D46, D47, D48, D49, D5, D50, D51, D52, D53, D54, D55, D56, D57, D58, D59, D6, D60, D61, D62, D63, D64, D65, D66, D7, D8, D9: moved to B.Cu
- S52: footprint ScottoKeebs_Hotswap:Hotswap_MX_1.50u -> ScottoKeebs_Hotswap:Hotswap_MX_1.00u
- S53: footprint ScottoKeebs_Hotswap:Hotswap_MX_1.00u -> ScottoKeebs_Hotswap:Hotswap_MX_1.50u
- U1: moved to F.Cu
- moved D7 139.2 mm to (186.7, 38.1), turned to 90 degrees
- moved D8 135.7 mm to (67.6, 57.1), turned to 90 degrees
- moved D40 131.9 mm to (367.7, 38.1), turned to 90 degrees
- moved D6 130.6 mm to (167.6, 38.1), turned to 90 degrees
- moved D1 129.5 mm to (72.4, 38.1), turned to 90 degrees
- moved D41 129.4 mm to (253.4, 57.1), turned to 90 degrees
- moved D9 127.9 mm to (91.4, 57.1), turned to 90 degrees
- moved D34 125.7 mm to (253.4, 38.1), turned to 90 degrees
- moved D5 124.5 mm to (148.6, 38.1), turned to 90 degrees
- moved D2 123.8 mm to (91.4, 38.1), turned to 90 degrees
- moved D39 123.6 mm to (348.6, 38.1), turned to 90 degrees
- moved D42 123.1 mm to (272.4, 57.1), turned to 90 degrees
- moved D4 121.3 mm to (129.5, 38.1), turned to 90 degrees
- moved D3 121.0 mm to (110.5, 38.1), turned to 90 degrees
- moved S53 119.2 mm to (366.7, 71.4)
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Connections:
- D48 pad 1: /Oath-66-Duo-Right/Col 0 -> /Oath-66-Duo-Right/Row 2
- D49 pad 1: /Oath-66-Duo-Right/Col 0 -> /Oath-66-Duo-Right/Row 2
- D50 pad 1: /Oath-66-Duo-Right/Col 0 -> /Oath-66-Duo-Right/Row 2
- D51 pad 1: /Oath-66-Duo-Right/Col 0 -> /Oath-66-Duo-Right/Row 2
- D52 pad 1: /Oath-66-Duo-Right/Col 0 -> /Oath-66-Duo-Right/Row 2
- D53 pad 1: /Oath-66-Duo-Right/Col 0 -> /Oath-66-Duo-Right/Row 2
- S62 pad 1: /Oath-66-Duo-Right/Col 2 -> /Oath-66-Duo-Right/Col 1
- U2 pad 12: /Oath-66-Duo-Right/Col 0 -> /Oath-66-Duo-Right/Row 2
Routing:
- net /Oath-66-Duo-Right/Col 1: track 0.00 -> 83.0 mm
- net /Oath-66-Duo-Left/Col 4: track 0.00 -> 82.9 mm
- net /Oath-66-Duo-Left/Col 6: track 0.00 -> 80.4 mm
- net /Oath-66-Duo-Left/Col 0: track 0.00 -> 80.2 mm
- net /Oath-66-Duo-Right/Col 6: track 0.00 -> 80.2 mm
- net /Oath-66-Duo-Right/Col 0: track 0.00 -> 80.2 mm
- net /Oath-66-Duo-Left/Col 3: track 0.00 -> 78.4 mm
- net /Oath-66-Duo-Right/Col 5: track 0.00 -> 76.2 mm
- net /Oath-66-Duo-Right/Col 4: track 0.00 -> 76.2 mm
- net /Oath-66-Duo-Right/Col 3: track 0.00 -> 76.2 mm
- net /Oath-66-Duo-Left/Col 2: track 0.00 -> 76.2 mm
- net /Oath-66-Duo-Left/Col 1: track 0.00 -> 76.2 mm
- net /Oath-66-Duo-Right/Col 2: track 0.00 -> 57.2 mm
- net /Oath-66-Duo-Left/Col 5: track 0.00 -> 57.2 mm
- net Net-(D63-A): track 0.00 -> 9.32 mm
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Other:
- board outline added: 379.1 x 99.1 mm

Commit message: PCB Updated
Routing:
- net /Oath-66-Duo-Left/Row 3: track 0.00 -> 169.7 mm, vias 0 -> 7
- net /Oath-66-Duo-Left/Row 1: track 0.00 -> 160.9 mm, vias 0 -> 7
- net /Oath-66-Duo-Left/Row 0: track 0.00 -> 160.9 mm, vias 0 -> 7
- net /Oath-66-Duo-Right/Col 0: track 80.2 -> 233.8 mm, vias 0 -> 1
- net /Oath-66-Duo-Left/Row 4: track 0.00 -> 152.6 mm, vias 0 -> 6
- net /Oath-66-Duo-Right/Row 3: track 0.00 -> 150.3 mm, vias 0 -> 8
- net /Oath-66-Duo-Right/Row 1: track 0.00 -> 149.4 mm, vias 0 -> 7
- net /Oath-66-Duo-Right/Row 0: track 0.00 -> 149.4 mm, vias 0 -> 7
- net /Oath-66-Duo-Right/Row 4: track 0.00 -> 148.5 mm, vias 0 -> 7
- net /Oath-66-Duo-Left/Row 2: track 0.00 -> 138.7 mm, vias 0 -> 6
- net /Oath-66-Duo-Right/Col 1: track 83.0 -> 217.5 mm, vias 0 -> 1
- net /Oath-66-Duo-Left/Col 6: track 80.4 -> 212.3 mm, vias 0 -> 1
- net /Oath-66-Duo-Right/Row 2: track 0.00 -> 127.3 mm, vias 0 -> 6
- net /Oath-66-Duo-Right/Col 2: track 57.2 -> 172.6 mm, vias 0 -> 1
- net /Oath-66-Duo-Left/Col 5: track 57.2 -> 168.4 mm, vias 0 -> 1
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
Commit message: PCB Updated
Parts:
- added REF**: MountingHole_2.5mm, MountingHole:MountingHole_2.5mm, F.Cu at (257.2, 100.0)
- added REF**: MountingHole_2.5mm, MountingHole:MountingHole_2.5mm, F.Cu at (376.2, 109.5)
- added REF**: MountingHole_2.5mm, MountingHole:MountingHole_2.5mm, F.Cu at (49.5, 109.5)
- added REF**: MountingHole_2.5mm, MountingHole:MountingHole_2.5mm, F.Cu at (171.4, 100.0)
- added REF**: MountingHole_2.5mm, MountingHole:MountingHole_2.5mm, F.Cu at (376.2, 33.3)
- added REF**: MountingHole_2.5mm, MountingHole:MountingHole_2.5mm, F.Cu at (52.4, 33.3)
Connections:
- U1 pad 10: /Oath-66-Duo-Left/Col 1 -> /Oath-66-Duo-Left/Row 3
- U1 pad 11: /Oath-66-Duo-Left/Col 2 -> /Oath-66-Duo-Left/Col 4
- U1 pad 12: /Oath-66-Duo-Left/Row 2 -> /Oath-66-Duo-Left/Row 4
- U1 pad 13: /Oath-66-Duo-Left/Col 4 -> /Oath-66-Duo-Left/Col 5
- U1 pad 14: /Oath-66-Duo-Left/Row 4 -> /Oath-66-Duo-Left/Col 6
- U1 pad 15: /Oath-66-Duo-Left/Col 3 -> /Oath-66-Duo-Left/Row 0
- U1 pad 16: /Oath-66-Duo-Left/Row 3 -> /Oath-66-Duo-Left/Col 0
- U1 pad 5: /Oath-66-Duo-Left/Col 5 -> /Oath-66-Duo-Left/Col 1
- U1 pad 6: /Oath-66-Duo-Left/Col 6 -> /Oath-66-Duo-Left/Row 1
- U1 pad 7: /Oath-66-Duo-Left/Row 0 -> /Oath-66-Duo-Left/Col 2
- U1 pad 8: /Oath-66-Duo-Left/Col 0 -> /Oath-66-Duo-Left/Row 2
- U1 pad 9: /Oath-66-Duo-Left/Row 1 -> /Oath-66-Duo-Left/Col 3
- U2 pad 10: /Oath-66-Duo-Right/Col 1 -> /Oath-66-Duo-Right/Row 0
- U2 pad 11: /Oath-66-Duo-Right/Col 2 -> /Oath-66-Duo-Right/Col 6
- U2 pad 12: /Oath-66-Duo-Right/Row 2 -> /Oath-66-Duo-Right/Col 5
- U2 pad 13: /Oath-66-Duo-Right/Col 4 -> /Oath-66-Duo-Right/Row 4
- U2 pad 14: /Oath-66-Duo-Right/Row 4 -> /Oath-66-Duo-Right/Col 4
- U2 pad 15: /Oath-66-Duo-Right/Col 3 -> /Oath-66-Duo-Right/Row 3
- U2 pad 16: /Oath-66-Duo-Right/Row 3 -> /Oath-66-Duo-Right/Col 3
- U2 pad 17: unconnected-(U2-A0/PF7-Pad17) -> /Oath-66-Duo-Right/Row 2
- U2 pad 18: unconnected-(U2-A1/PF6-Pad18) -> /Oath-66-Duo-Right/Col 2
- U2 pad 19: unconnected-(U2-A2/PF5-Pad19) -> /Oath-66-Duo-Right/Row 1
- U2 pad 20: unconnected-(U2-A3/PF4-Pad20) -> /Oath-66-Duo-Right/Col 1
- U2 pad 5: /Oath-66-Duo-Right/Col 5 -> unconnected-(U2-2/PD1-Pad5)
- U2 pad 6: /Oath-66-Duo-Right/Col 6 -> unconnected-(U2-3/PD0-Pad6)
- U2 pad 7: /Oath-66-Duo-Right/Row 0 -> unconnected-(U2-4/PD4-Pad7)
- U2 pad 8: /Oath-66-Duo-Right/Col 0 -> unconnected-(U2-5/PC6-Pad8)
- U2 pad 9: /Oath-66-Duo-Right/Row 1 -> /Oath-66-Duo-Right/Col 0
Routing:
- net /Oath-66-Duo-Left/Col 4: track 178.5 -> 259.4 mm, vias 1 -> 3
- net /Oath-66-Duo-Right/Row 4: track 148.5 -> 229.3 mm, vias 7 -> 9
- net /Oath-66-Duo-Right/Col 4: track 153.6 -> 234.3 mm, vias 1 -> 3
- net /Oath-66-Duo-Left/Row 4: track 152.6 -> 232.6 mm, vias 6 -> 8
- net /Oath-66-Duo-Right/Row 3: track 150.3 -> 216.6 mm, vias 8 -> 10
- net /Oath-66-Duo-Right/Col 3: track 172.6 -> 238.6 mm, vias 1 -> 3
- net /Oath-66-Duo-Left/Col 3: track 155.8 -> 216.8 mm, vias 1 -> 3
- net /Oath-66-Duo-Left/Row 3: track 169.7 -> 228.5 mm, vias 7 -> 9
- net /Oath-66-Duo-Right/Row 2: track 127.3 -> 180.6 mm, vias 6 -> 8
- net /Oath-66-Duo-Right/Col 2: track 172.6 -> 225.7 mm, vias 1 -> 3
- net /Oath-66-Duo-Left/Col 2: track 134.5 -> 182.8 mm, vias 1 -> 3
- net /Oath-66-Duo-Left/Row 2: track 138.7 -> 186.2 mm, vias 6 -> 8
- net /Oath-66-Duo-Left/Col 1: track 115.5 -> 155.1 mm, vias 1 -> 3
- net /Oath-66-Duo-Right/Row 1: track 149.4 -> 188.9 mm, vias 7 -> 9
- net /Oath-66-Duo-Right/Col 1: track 217.5 -> 256.9 mm, vias 1 -> 3
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
Commit message: PCB Updated
Parts:
- added REF**: MountingHole_2.5mm, MountingHole:MountingHole_2.5mm, F.Cu at (314.3, 61.9)
- added REF**: MountingHole_2.5mm, MountingHole:MountingHole_2.5mm, F.Cu at (171.4, 42.9)
- added REF**: MountingHole_2.5mm, MountingHole:MountingHole_2.5mm, F.Cu at (114.3, 61.9)
- added REF**: MountingHole_2.5mm, MountingHole:MountingHole_2.5mm, F.Cu at (257.2, 42.9)
- moved REF** 3.72 mm to (52.4, 107.2)
Connections:
- U2 pad 10: /Oath-66-Duo-Right/Row 0 -> /Oath-66-Duo-Right/Col 0
- U2 pad 12: /Oath-66-Duo-Right/Col 5 -> /Oath-66-Duo-Right/Row 0
- U2 pad 14: /Oath-66-Duo-Right/Col 4 -> /Oath-66-Duo-Right/Col 2
- U2 pad 18: /Oath-66-Duo-Right/Col 2 -> /Oath-66-Duo-Right/Col 4
- U2 pad 20: /Oath-66-Duo-Right/Col 1 -> /Oath-66-Duo-Right/Col 5
- U2 pad 9: /Oath-66-Duo-Right/Col 0 -> /Oath-66-Duo-Right/Col 1
Routing:
- net /Oath-66-Duo-Right/Col 4: track 234.3 -> 202.4 mm
- net /Oath-66-Duo-Right/Col 2: track 225.7 -> 256.6 mm
- net /Oath-66-Duo-Right/Col 1: track 256.9 -> 238.3 mm, vias 3 -> 2
- net /Oath-66-Duo-Right/Row 0: track 158.8 -> 173.3 mm
- net /Oath-66-Duo-Right/Col 6: track 147.9 -> 134.2 mm, vias 2 -> 1
- net /Oath-66-Duo-Right/Col 5: track 161.4 -> 174.4 mm, vias 2 -> 1
- net /Oath-66-Duo-Right/Col 0: track 243.0 -> 251.4 mm, vias 1 -> 2
- net /Oath-66-Duo-Right/Row 4: track 229.3 -> 222.8 mm
- net /Oath-66-Duo-Right/Col 3: track 238.6 -> 233.1 mm
- net /Oath-66-Duo-Left/Row 1: track 199.8 -> 204.9 mm
- net /Oath-66-Duo-Left/Row 0: track 170.2 -> 175.4 mm
- net /Oath-66-Duo-Right/Row 1: track 188.9 -> 194.1 mm
- net /Oath-66-Duo-Right/Row 2: track 180.6 -> 176.4 mm
- net /Oath-66-Duo-Left/Row 4: track 232.6 -> 236.4 mm
- net /Oath-66-Duo-Right/Row 3: track 216.6 -> 212.9 mm
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
Commit message: Schematic and PCB Updated
Parts:
- removed the REF** at (257.2, 100.0)
- removed the REF** at (376.2, 33.3)
- removed the REF** at (314.3, 61.9)
- removed the REF** at (52.4, 33.3)
- removed the REF** at (376.2, 109.5)
- removed the REF** at (52.4, 107.2)
- removed the REF** at (171.4, 42.9)
- removed the REF** at (114.3, 61.9)
- removed the REF** at (257.2, 42.9)
- removed the REF** at (171.4, 100.0)
- added H1: Mounting_Hole, MountingHole:MountingHole_2.5mm, F.Cu at (52.4, 33.3)
- added H10: Mounting_Hole, MountingHole:MountingHole_2.5mm, F.Cu at (376.2, 109.5)
- added H2: Mounting_Hole, MountingHole:MountingHole_2.5mm, F.Cu at (171.4, 42.9)
- added H3: Mounting_Hole, MountingHole:MountingHole_2.5mm, F.Cu at (114.3, 61.9)
- added H4: Mounting_Hole, MountingHole:MountingHole_2.5mm, F.Cu at (52.4, 107.2)
- added H5: Mounting_Hole, MountingHole:MountingHole_2.5mm, F.Cu at (171.4, 100.0)
- added H6: Mounting_Hole, MountingHole:MountingHole_2.5mm, F.Cu at (376.2, 33.3)
- added H7: Mounting_Hole, MountingHole:MountingHole_2.5mm, F.Cu at (257.2, 42.9)
- added H8: Mounting_Hole, MountingHole:MountingHole_2.5mm, F.Cu at (314.3, 61.9)
- added H9: Mounting_Hole, MountingHole:MountingHole_2.5mm, F.Cu at (257.2, 100.0)
- added J1: Conn_01x02, Connector_JST:JST_PH_S2B-PH-K_1x02_P2.00mm_Horizontal, F.Cu at (32.9, 79.5)
- added J2: Conn_01x02, Connector_JST:JST_PH_S2B-PH-K_1x02_P2.00mm_Horizontal, F.Cu at (394.8, 80.4)
- added PSW1: ~, MyLibrary:MSK_1134_3PIN_2H, F.Cu at (40.0, 65.7)
- added PSW2: ~, MyLibrary:MSK_1134_3PIN_2H, F.Cu at (388.6, 65.6)
- added RSW1: ~, MyLibrary:Tactile_Switch_3_6_2.5mm, F.Cu at (28.6, 65.7)
- added RSW2: ~, MyLibrary:Tactile_Switch_3_6_2.5mm, F.Cu at (399.6, 65.2)
Connections:
- net /Oath-66-Duo-Left/Col 0 renamed /Oath-66-Duo-Left/COL0_L
- net /Oath-66-Duo-Left/Col 1 renamed /Oath-66-Duo-Left/COL1_L
- net /Oath-66-Duo-Left/Col 2 renamed /Oath-66-Duo-Left/COL2_L
- net /Oath-66-Duo-Left/Col 3 renamed /Oath-66-Duo-Left/COL3_L
- net /Oath-66-Duo-Left/Col 4 renamed /Oath-66-Duo-Left/COL4_L
- net /Oath-66-Duo-Left/Col 5 renamed /Oath-66-Duo-Left/COL5_L
- net /Oath-66-Duo-Left/Col 6 renamed /Oath-66-Duo-Left/COL6_L
- net /Oath-66-Duo-Left/Row 0 renamed /Oath-66-Duo-Left/ROW0_L
- net /Oath-66-Duo-Left/Row 1 renamed /Oath-66-Duo-Left/ROW1_L
- net /Oath-66-Duo-Left/Row 2 renamed /Oath-66-Duo-Left/ROW2_L
- net /Oath-66-Duo-Left/Row 3 renamed /Oath-66-Duo-Left/ROW3_L
- net /Oath-66-Duo-Left/Row 4 renamed /Oath-66-Duo-Left/ROW4_L
- net /Oath-66-Duo-Right/Col 0 renamed /Oath-66-Duo-Right/COL0_R
- net /Oath-66-Duo-Right/Col 1 renamed /Oath-66-Duo-Right/COL1_R
- net /Oath-66-Duo-Right/Col 2 renamed /Oath-66-Duo-Right/COL2_R
- net /Oath-66-Duo-Right/Col 3 renamed /Oath-66-Duo-Right/COL3_R
- net /Oath-66-Duo-Right/Col 4 renamed /Oath-66-Duo-Right/COL4_R
- net /Oath-66-Duo-Right/Col 5 renamed /Oath-66-Duo-Right/COL5_R
- net /Oath-66-Duo-Right/Col 6 renamed /Oath-66-Duo-Right/COL6_R
- net /Oath-66-Duo-Right/Row 0 renamed /Oath-66-Duo-Right/ROW0_R
- net /Oath-66-Duo-Right/Row 1 renamed /Oath-66-Duo-Right/ROW1_R
- net /Oath-66-Duo-Right/Row 2 renamed /Oath-66-Duo-Right/ROW2_R
- net /Oath-66-Duo-Right/Row 3 renamed /Oath-66-Duo-Right/ROW3_R
- net /Oath-66-Duo-Right/Row 4 renamed /Oath-66-Duo-Right/ROW4_R
- U1 pad 21: unconnected-(U1-VCC-Pad21) -> /Oath-66-Duo-Left/BAT+_L
- U1 pad 22: unconnected-(U1-RST-Pad22) -> /Oath-66-Duo-Left/RST_L
- U1 pad 3: unconnected-(U1-GND-Pad3) -> /Oath-66-Duo-Left/GND_L
- U1 pad 4: unconnected-(U1-GND-Pad4) -> /Oath-66-Duo-Left/GND_L
- U2 pad 21: unconnected-(U2-VCC-Pad21) -> /Oath-66-Duo-Right/BAT+_R
- U2 pad 22: unconnected-(U2-RST-Pad22) -> /Oath-66-Duo-Right/RST_R
- U2 pad 3: unconnected-(U2-GND-Pad3) -> /Oath-66-Duo-Right/GND_R
- U2 pad 4: unconnected-(U2-GND-Pad4) -> /Oath-66-Duo-Right/GND_R

Commit message: PCB Routing Finished
Parts:
- J1, J2: value Conn_01x02 -> Connector_PH2.0_2Pin_Horizontal; footprint Connector_JST:JST_PH_S2B-PH-K_1x02_P2.00mm_Horizontal -> Connector_JST:JST_GH_SM02B-GHS-TB_1x02-1MP_P1.25mm_Horizontal
- PSW1, PSW2: footprint MyLibrary:MSK_1134_3PIN_2H -> MyLibrary:MSK_1134_3Pin_2H
- moved PSW1 11.1 mm to (31.6, 73.0), turned to 90 degrees
- moved RSW2 11.1 mm to (388.7, 63.0), turned to 180 degrees
- moved J1 10.6 mm to (41.1, 73.0)
- moved J2 8.23 mm to (398.3, 73.0)
- moved PSW2 7.40 mm to (388.7, 73.0), turned to 90 degrees
- moved RSW1 4.04 mm to (31.6, 63.0), turned to 180 degrees
Connections:
- U1 pad 23: unconnected-(U1-GND-Pad23) -> /Oath-66-Duo-Left/GND_L
- U2 pad 23: unconnected-(U2-GND-Pad23) -> /Oath-66-Duo-Right/GND_R
Routing:
- net /Oath-66-Duo-Left/GND_L: track 0.00 -> 79.7 mm, vias 0 -> 3
- net /Oath-66-Duo-Right/GND_R: track 0.00 -> 79.4 mm, vias 0 -> 3
- net /Oath-66-Duo-Right/BAT+_R: track 0.00 -> 49.8 mm, vias 0 -> 1
- net /Oath-66-Duo-Left/BAT+_L: track 0.00 -> 49.1 mm
- net /Oath-66-Duo-Right/RST_R: track 0.00 -> 44.9 mm, vias 0 -> 1
- net /Oath-66-Duo-Left/RST_L: track 0.00 -> 42.8 mm, vias 0 -> 2
- net /Oath-66-Duo-Right/VBAT_R: track 0.00 -> 6.19 mm
- net /Oath-66-Duo-Left/VBAT_L: track 0.00 -> 6.19 mm
- net /Oath-66-Duo-Right/COL5_R: track 174.4 -> 173.0 mm
- added copper zone on B.Cu, net /Oath-66-Duo-Left/GND_L
- added copper zone on F.Cu, net /Oath-66-Duo-Left/GND_L
- added copper zone on B.Cu, net /Oath-66-Duo-Right/GND_R
- added copper zone on F.Cu, net /Oath-66-Duo-Right/GND_R

Commit message: Bug Fixed
Parts:
- U1, U2: value Arduino_Pro_Micro -> nice_nano; footprint ScottoKeebs_MCU:Arduino_Pro_Micro -> PCM_marbastlib-xp-promicroish:nice_nano_AH_USBup
Connections:
- net /Oath-66-Duo-Left/COL1_L renamed COL1_L
- net /Oath-66-Duo-Left/COL2_L renamed COL2_L
- net /Oath-66-Duo-Left/COL3_L renamed COL3_L
- net /Oath-66-Duo-Left/COL4_L renamed COL4_L
- net /Oath-66-Duo-Left/ROW1_L renamed ROW1_L
- net /Oath-66-Duo-Left/ROW2_L renamed ROW2_L
- net /Oath-66-Duo-Left/ROW3_L renamed ROW3_L
- net /Oath-66-Duo-Left/ROW4_L renamed ROW4_L
- net /Oath-66-Duo-Left/VBAT_L renamed VBAT_L
- net /Oath-66-Duo-Right/COL0_R renamed COL0_R
- net /Oath-66-Duo-Right/COL1_R renamed COL1_R
- net /Oath-66-Duo-Right/COL6_R renamed COL6_R
- net /Oath-66-Duo-Right/ROW0_R renamed ROW0_R
- net /Oath-66-Duo-Right/VBAT_R renamed VBAT_R
- D1 pad 1: /Oath-66-Duo-Left/ROW0_L -> ROW0_L
- D2 pad 1: /Oath-66-Duo-Left/ROW0_L -> ROW0_L
- D3 pad 1: /Oath-66-Duo-Left/ROW0_L -> ROW0_L
- D4 pad 1: /Oath-66-Duo-Left/ROW0_L -> ROW0_L
- D41 pad 1: /Oath-66-Duo-Right/ROW1_R -> ROW1_R
- D42 pad 1: /Oath-66-Duo-Right/ROW1_R -> ROW1_R
- D43 pad 1: /Oath-66-Duo-Right/ROW1_R -> ROW1_R
- D44 pad 1: /Oath-66-Duo-Right/ROW1_R -> ROW1_R
- D45 pad 1: /Oath-66-Duo-Right/ROW1_R -> ROW1_R
- D46 pad 1: /Oath-66-Duo-Right/ROW1_R -> ROW1_R
- D47 pad 1: /Oath-66-Duo-Right/ROW1_R -> ROW1_R
- D48 pad 1: /Oath-66-Duo-Right/ROW2_R -> ROW2_R
- D49 pad 1: /Oath-66-Duo-Right/ROW2_R -> ROW2_R
- D5 pad 1: /Oath-66-Duo-Left/ROW0_L -> ROW0_L
- D50 pad 1: /Oath-66-Duo-Right/ROW2_R -> ROW2_R
- D51 pad 1: /Oath-66-Duo-Right/ROW2_R -> ROW2_R
- D52 pad 1: /Oath-66-Duo-Right/ROW2_R -> ROW2_R
- D53 pad 1: /Oath-66-Duo-Right/ROW2_R -> ROW2_R
- D54 pad 1: /Oath-66-Duo-Right/ROW3_R -> ROW3_R
- D55 pad 1: /Oath-66-Duo-Right/ROW3_R -> ROW3_R
- D56 pad 1: /Oath-66-Duo-Right/ROW3_R -> ROW3_R
- D57 pad 1: /Oath-66-Duo-Right/ROW3_R -> ROW3_R
- D58 pad 1: /Oath-66-Duo-Right/ROW3_R -> ROW3_R
- D59 pad 1: /Oath-66-Duo-Right/ROW3_R -> ROW3_R
- D6 pad 1: /Oath-66-Duo-Left/ROW0_L -> ROW0_L
- D60 pad 1: /Oath-66-Duo-Right/ROW3_R -> ROW3_R
- D61 pad 1: /Oath-66-Duo-Right/ROW4_R -> ROW4_R
- D62 pad 1: /Oath-66-Duo-Right/ROW4_R -> ROW4_R
- D63 pad 1: /Oath-66-Duo-Right/ROW4_R -> ROW4_R
- D64 pad 1: /Oath-66-Duo-Right/ROW4_R -> ROW4_R
- D65 pad 1: /Oath-66-Duo-Right/ROW4_R -> ROW4_R
- D66 pad 1: /Oath-66-Duo-Right/ROW4_R -> ROW4_R
- D7 pad 1: /Oath-66-Duo-Left/ROW0_L -> ROW0_L
- J1 pad 2: /Oath-66-Duo-Left/GND_L -> GND_L
- J2 pad 2: /Oath-66-Duo-Right/GND_R -> GND_R
- PSW1 pad 2: /Oath-66-Duo-Left/BAT+_L -> BAT+_L
- PSW2 pad 2: /Oath-66-Duo-Right/BAT+_R -> BAT+_R
- RSW1 pad 1: /Oath-66-Duo-Left/RST_L -> RST_L
- RSW1 pad 2: /Oath-66-Duo-Left/GND_L -> GND_L
- RSW2 pad 1: /Oath-66-Duo-Right/RST_R -> RST_R
- RSW2 pad 2: /Oath-66-Duo-Right/GND_R -> GND_R
- S1 pad 1: /Oath-66-Duo-Left/COL0_L -> COL0_L
- S13 pad 1: /Oath-66-Duo-Left/COL5_L -> COL5_L
- S14 pad 1: /Oath-66-Duo-Left/COL6_L -> COL6_L
- S15 pad 1: /Oath-66-Duo-Left/COL0_L -> COL0_L
- S20 pad 1: /Oath-66-Duo-Left/COL5_L -> COL5_L
- S21 pad 1: /Oath-66-Duo-Left/COL0_L -> COL0_L
- S26 pad 1: /Oath-66-Duo-Left/COL5_L -> COL5_L
- S27 pad 1: /Oath-66-Duo-Left/COL6_L -> COL6_L
- S28 pad 1: /Oath-66-Duo-Left/COL0_L -> COL0_L
- S33 pad 1: /Oath-66-Duo-Left/COL6_L -> COL6_L
- S36 pad 1: /Oath-66-Duo-Right/COL2_R -> COL2_R
- S37 pad 1: /Oath-66-Duo-Right/COL3_R -> COL3_R
- S38 pad 1: /Oath-66-Duo-Right/COL4_R -> COL4_R
- S39 pad 1: /Oath-66-Duo-Right/COL5_R -> COL5_R
- S43 pad 1: /Oath-66-Duo-Right/COL2_R -> COL2_R
- S44 pad 1: /Oath-66-Duo-Right/COL3_R -> COL3_R
- S45 pad 1: /Oath-66-Duo-Right/COL4_R -> COL4_R
- S46 pad 1: /Oath-66-Duo-Right/COL5_R -> COL5_R
- S49 pad 1: /Oath-66-Duo-Right/COL2_R -> COL2_R
- S50 pad 1: /Oath-66-Duo-Right/COL3_R -> COL3_R
- S51 pad 1: /Oath-66-Duo-Right/COL4_R -> COL4_R
- S52 pad 1: /Oath-66-Duo-Right/COL5_R -> COL5_R
- S56 pad 1: /Oath-66-Duo-Right/COL2_R -> COL2_R
- S57 pad 1: /Oath-66-Duo-Right/COL3_R -> COL3_R
- S58 pad 1: /Oath-66-Duo-Right/COL4_R -> COL4_R
- S59 pad 1: /Oath-66-Duo-Right/COL5_R -> COL5_R
- S6 pad 1: /Oath-66-Duo-Left/COL5_L -> COL5_L
- S63 pad 1: /Oath-66-Duo-Right/COL3_R -> COL3_R
- S64 pad 1: /Oath-66-Duo-Right/COL4_R -> COL4_R
- S65 pad 1: /Oath-66-Duo-Right/COL5_R -> COL5_R
- S7 pad 1: /Oath-66-Duo-Left/COL6_L -> COL6_L
- S8 pad 1: /Oath-66-Duo-Left/COL0_L -> COL0_L
- U1 pad 13: /Oath-66-Duo-Left/COL5_L -> unconnected-(U1-BAT+-Pad13)
- U1 pad 14: /Oath-66-Duo-Left/COL6_L -> GND_L
- U1 pad 15: /Oath-66-Duo-Left/ROW0_L -> RST_L
- U1 pad 16: /Oath-66-Duo-Left/COL0_L -> unconnected-(U1-3V3-Pad16)
- U1 pad 21: /Oath-66-Duo-Left/BAT+_L -> COL0_L
- U1 pad 22: /Oath-66-Duo-Left/RST_L -> ROW0_L
- U1 pad 23: /Oath-66-Duo-Left/GND_L -> COL6_L
- U1 pad 24: unconnected-(U1-RAW-Pad24) -> COL5_L
- U1 pad 3: /Oath-66-Duo-Left/GND_L -> GND_L
- U1 pad 4: /Oath-66-Duo-Left/GND_L -> GND_L
- U2 pad 13: /Oath-66-Duo-Right/ROW4_R -> unconnected-(U2-BAT+-Pad13)
- U2 pad 14: /Oath-66-Duo-Right/COL2_R -> GND_R
- U2 pad 15: /Oath-66-Duo-Right/ROW3_R -> RST_R
- U2 pad 16: /Oath-66-Duo-Right/COL3_R -> unconnected-(U2-3V3-Pad16)
- U2 pad 17: /Oath-66-Duo-Right/ROW2_R -> COL5_R
- U2 pad 18: /Oath-66-Duo-Right/COL4_R -> ROW1_R
- U2 pad 19: /Oath-66-Duo-Right/ROW1_R -> COL4_R
- U2 pad 20: /Oath-66-Duo-Right/COL5_R -> ROW2_R
- U2 pad 21: /Oath-66-Duo-Right/BAT+_R -> COL3_R
- U2 pad 22: /Oath-66-Duo-Right/RST_R -> ROW3_R
- U2 pad 23: /Oath-66-Duo-Right/GND_R -> COL2_R
- U2 pad 24: unconnected-(U2-RAW-Pad24) -> ROW4_R
- U2 pad 3: /Oath-66-Duo-Right/GND_R -> GND_R
- U2 pad 4: /Oath-66-Duo-Right/GND_R -> GND_R
Routing:
- net /Oath-66-Duo-Right/COL2_R: track 256.6 -> 0.00 mm, vias 3 -> 0
- net COL2_R: track 0.00 -> 254.8 mm, vias 0 -> 3
- net /Oath-66-Duo-Left/COL6_L: track 245.9 -> 0.00 mm, vias 2 -> 0
- net COL6_L: track 0.00 -> 245.5 mm, vias 0 -> 2
- net /Oath-66-Duo-Right/COL3_R: track 233.1 -> 0.00 mm, vias 3 -> 0
- net COL3_R: track 0.00 -> 229.6 mm, vias 0 -> 3
- net /Oath-66-Duo-Right/ROW4_R: track 222.8 -> 0.00 mm, vias 9 -> 0
- net ROW4_R: track 0.00 -> 222.7 mm, vias 0 -> 9
- net /Oath-66-Duo-Right/ROW3_R: track 212.9 -> 0.00 mm, vias 10 -> 0
- net ROW3_R: track 0.00 -> 210.0 mm, vias 0 -> 10
- net /Oath-66-Duo-Right/COL4_R: track 202.4 -> 0.00 mm, vias 3 -> 0
- net COL5_L: track 0.00 -> 199.8 mm, vias 0 -> 2
- net /Oath-66-Duo-Left/COL5_L: track 199.8 -> 0.00 mm, vias 2 -> 0
- net COL4_R: track 0.00 -> 197.8 mm, vias 0 -> 3
- net /Oath-66-Duo-Right/ROW1_R: track 194.1 -> 0.00 mm, vias 9 -> 0
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- added copper zone on B.Cu, net GND_L
- added copper zone on F.Cu, net GND_L
- added copper zone on B.Cu, net GND_R
- added copper zone on F.Cu, net GND_R
- removed copper zone on B.Cu, net /Oath-66-Duo-Left/GND_L
- removed copper zone on F.Cu, net /Oath-66-Duo-Left/GND_L
- removed copper zone on B.Cu, net /Oath-66-Duo-Right/GND_R
- removed copper zone on F.Cu, net /Oath-66-Duo-Right/GND_R
