File: PCB/Oath-66-Duo.kicad_pcb (KiCad board)
At the start: 2 copper layers, 379.1 x 99.1 mm, 154 parts, among them J1 Connector_PH2.0_2Pin_Horizont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, J2 Connector_PH2.0_2Pin_Horizont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, U1 nice_nano, U2 nice_nano

Commit message: Prepared for production
Parts:
- moved D35 30.0 mm to (242.4, 38.1)
- moved D42 30.0 mm to (242.4, 57.1)
- moved D48 30.0 mm to (242.4, 76.2)
- moved D55 30.0 mm to (242.4, 95.2)
- moved D34 30.0 mm to (223.4, 38.1)
- moved D36 30.0 mm to (261.5, 38.1)
- moved D37 30.0 mm to (280.5, 38.1)
- moved D38 30.0 mm to (299.6, 38.1)
- moved D39 30.0 mm to (318.6, 38.1)
- moved D40 30.0 mm to (337.7, 38.1)
- moved D41 30.0 mm to (223.4, 57.1)
- moved D43 30.0 mm to (261.5, 57.1)
- moved D44 30.0 mm to (280.5, 57.1)
- moved D45 30.0 mm to (299.6, 57.1)
- moved D46 30.0 mm to (318.6, 57.1)
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Other:
- board size 379.1 x 99.1 mm -> 349.1 x 99.1 mm

Commit message: Battery Connector Updated
Parts:
- J1, J2: value Connector_PH2.0_2Pin_Horizontal -> GH1.25 Battery Connector
Connections:
- J1 pad 1: VBAT_L -> GND_L
- J1 pad 2: GND_L -> VBAT_L
- J2 pad 1: VBAT_R -> GND_R
- J2 pad 2: GND_R -> VBAT_R
Routing:
- net VBAT_L: track 6.19 -> 19.0 mm
- net VBAT_R: track 6.19 -> 17.2 mm
- net GND_L: track 104.6 -> 105.5 mm
- net GND_R: track 105.7 -> 106.2 mm
Changed lines of the file:
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@@
 		(tags "connector JST GH horizontal")
 		(property "Reference" "J1"
-			(at 0 4.64625 0)
+			(at 1.781 4.2335 0)
 			(layer "F.SilkS")
 			(effects
@@
 			)
 		)
-		(property "Value" "Connector_PH2.0_2Pin_Horizontal"
+		(property "Value" "GH1.25 Battery Connector"
 			(at 0 3.9 0)
 			(layer "F.Fab")
@@
 			(layers "F.Cu" "F.Mask" "F.Paste")
 			(roundrect_rratio 0.25)
-			(net 83 "VBAT_L")
+			(net 84 "GND_L")
 			(pinfunction "Pin_1")
 			(pintype "passive")
@@
 			(layers "F.Cu" "F.Mask" "F.Paste")
 			(roundrect_rratio 0.25)
-			(net 84 "GND_L")
+			(net 83 "VBAT_L")
 			(pinfunction "Pin_2")
 			(pintype "passive")
@@
 			)
 		)
-		(property "Value" "Connector_PH2.0_2Pin_Horizontal"
+		(property "Value" "GH1.25 Battery Connector"
 			(at 0 3.9 0)
 			(layer "F.Fab")
@@
 			(layers "F.Cu" "F.Mask" "F.Paste")
 			(roundrect_rratio 0.25)
-			(net 86 "VBAT_R")
+			(net 85 "GND_R")
 			(pinfunction "Pin_1")
 			(pintype "passive")
@@
 			(layers "F.Cu" "F.Mask" "F.Paste")
 			(roundrect_rratio 0.25)
-			(net 85 "GND_R")
+			(net 86 "VBAT_R")
 			(pinfunction "Pin_2")
 			(pintype "passive")
@@
 	)
 	(segment
+		(start 37.592 77.47)
+		(end 41.034 77.47)
+		(width 0.508)
+		(layer "F.Cu")
+		(net 83)
+	)
+	(segment
+		(start 41.034 77.47)
+		(end 41.77 76.734)
+		(width 0.508)
+		(layer "F.Cu")
+		(net 83)
+	)
+	(segment
+		(start 41.77 76.734)
+		(end 41.77 71.1325)
+		(width 0.508)
+		(layer "F.Cu")
+		(net 83)
+	)
+	(segment
+		(start 36.83 71.628)
+		(end 36.83 76.708)
+		(width 0.508)
+		(layer "F.Cu")
+		(net 83)
+	)
+	(segment
+		(start 35.6845 70.4825)
+		(end 36.83 71.628)
+		(width 0.508)
+		(layer "F.Cu")
+		(net 83)
+	)
+	(segment
 		(start 34.595 70.4825)
-		(end 39.87 70.4825)
+		(end 35.6845 70.4825)
 		(width 0.508)
 		(layer "F.Cu")
@@
 	)
 	(segment
-		(start 39.87 70.4825)
-		(end 40.52 71.1325)
+		(start 36.83 76.708)
+		(end 37.592 77.47)
 		(width 0.508)
 		(layer "F.Cu")
@@
 	)
 	(segment
-		(start 41.77 37.084)
-		(end 41.77 71.1325)
+		(start 40.52 67.176)
+		(end 40.52 71.1325)
+		(width 0.508)
+		(layer "F.Cu")
+		(net 84)
+	)
+	(segment
+		(start 41.656 37.338)
+		(end 41.656 66.04)
+		(width 0.508)
+		(layer "F.Cu")
+		(net 84)
+	)
+	(segment
+		(start 41.656 66.04)
+		(end 40.52 67.176)
 		(width 0.508)
 		(layer "F.Cu")
@@
 	)
 	(via
-		(at 41.77 37.084)
+		(at 41.656 37.338)
 		(size 0.6)
 		(drill 0.3)
@@
 	)
 	(segment
-		(start 38.9125 25.0825)
-		(end 28.41625 25.0825)
+		(start 39.0525 25.0825)
+		(end 28.115 25.0825)
 		(width 0.508)
 		(layer "B.Cu")
@@
 	)
 	(segment
-		(start 41.77 37.084)
-		(end 41.77 27.94)
+		(start 41.656 37.338)
+		(end 41.656 27.686)
 		(width 0.508)
 		(layer "B.Cu")
@@
 	)
 	(segment
-		(start 41.77 27.94)
-		(end 38.9125 25.0825)
+		(start 41.656 27.686)
+		(end 39.0525 25.0825)
 		(width 0.508)
 		(layer "B.Cu")
@@
 	)
 	(segment
+		(start 367.674936 66.665064)
+		(end 367.674936 71.1325)
+		(width 0.508)
+		(layer "F.Cu")
+		(net 85)
+	)
+	(segment
 		(start 355.318 60.198)
 		(end 354.999936 60.516064)
@@
 	)
 	(segment
+		(start 368.924936 64.653064)
+		(end 368.924936 65.415064)
+		(width 0.508)
+		(layer "F.Cu")
+		(net 85)
+	)
+	(segment
+		(start 368.924936 65.415064)
+		(end 367.674936 66.665064)
+		(width 0.508)
+		(layer "F.Cu")
+		(net 85)
+	)
+	(segment
 		(start 364.1445 32.7025)
 		(end 365.478 34.036)
@@
 		(net 85)
 	)
-	(segment
-		(start 368.924936 64.77)
-		(end 368.924936 71.1325)
-		(width 0.508)
-		(layer "F.Cu")
-		(net 85)
-	)
 	(via
 		(at 355.318 60.198)
@@
 	)
 	(via
-		(at 368.924936 64.77)
+		(at 368.924936 64.653064)
 		(size 0.6)
 		(drill 0.3)
@@
 	)
 	(segment
-		(start 368.924936 27.576936)
-		(end 366.4305 25.0825)
-		(width 0.508)
-		(layer "B.Cu")
-		(net 85)
-	)
-	(segment
 		(start 364.716 49.53)
 		(end 365.478 48.768)
@@
 	)
 	(segment
+		(start 365.478 48.768)
+		(end 365.478 34.036)
+		(width 0.254)
+		(layer "B.Cu")
+		(net 85)
+	)
+	(segment
 		(start 366.4305 25.0825)
 		(end 355.269936 25.0825)
@@
 	)
 	(segment
-		(start 368.924936 64.77)
+		(start 368.924936 64.653064)
 		(end 368.924936 27.576936)
 		(width 0.508)
@@
 	)
 	(segment
-		(start 365.478 48.768)
-		(end 365.478 34.036)
-		(width 0.254)
+		(start 368.924936 27.576936)
+		(end 366.4305 25.0825)
+		(width 0.508)
 		(layer "B.Cu")
 		(net 85)
@@
 	)
 	(segment
-		(start 367.024936 70.4825)
-		(end 367.674936 71.1325)
+		(start 363.982 76.2)
+		(end 364.744 76.962)
+		(width 0.508)
+		(layer "F.Cu")
+		(net 86)
+	)
+	(segment
+		(start 364.744 76.962)
+		(end 368.046 76.962)
 		(width 0.508)
 		(layer "F.Cu")
@@
 	(segment
 		(start 361.749936 70.4825)
-		(end 367.024936 70.4825)
+		(end 363.982 72.714564)
+		(width 0.508)
+		(layer "F.Cu")
+		(net 86)
+	)
+	(segment
+		(start 368.046 76.962)
+		(end 368.924936 76.083064)
+		(width 0.508)
+		(layer "F.Cu")
+		(net 86)
+	)
+	(segment
+		(start 363.982 72.714564)
+		(end 363.982 76.2)
+		(width 0.508)
+		(layer "F.Cu")
+		(net 86)
+	)
+	(segment
+		(start 368.924936 76.083064)
+		(end 368.924936 71.1325)
 		(width 0.508)
 		(layer "F.Cu")

Commit message: PCB Updated
Parts:
- turned REF** to -90 degrees
- turned REF** to 90 degrees
- turned REF** to 180 degrees (x2)
Routing:
- net ROW3_L: track 234.4 -> 229.2 mm, vias 9 -> 7
- net ROW4_L: track 235.9 -> 231.9 mm
- net ROW3_R: track 210.0 -> 213.2 mm, vias 10 -> 9
- net COL6_L: track 245.5 -> 243.3 mm
- net ROW4_R: track 222.7 -> 220.8 mm, vias 9 -> 8
- net COL1_R: track 238.3 -> 239.7 mm
- net COL4_L: track 260.1 -> 261.5 mm
